File: pcb/pcb-v5/pcb-v5.sch (KiCad schematic (older format))
At the start: 18 parts, among them J1 Conn_01x05_Female, J2 Conn_01x05_Female, J3 Conn_01x05_Female, J4 Conn_01x05_Male, Q1 2N7002, SW1 G71Y, SW2 G71Y, SW3 G71Y, U1 AMS1117-3.3

Commit message: PCB-V5 update
Updated after meeting
Parts:
- added e1: 02x06_pad, pcb-v5:02x06_pad, symbol sensOCampus:02x06_pad
Connections:
- no-connect marks 20 -> 30
Changed lines of the file:
@@
 Wire Notes Line
 	6300 1650 6300 450
+$Comp
+L sensOCampus:02x06_pad e1
+U 1 1 601241B4
+P 6300 5100
+F 0 "e1" H 6375 5575 50  0000 C CNN
+F 1 "02x06_pad" H 6375 5484 50  0000 C CNN
+F 2 "pcb-v5:02x06_pad" H 6300 5100 50  0001 C CNN
+F 3 "" H 6300 5100 50  0001 C CNN
+	1    6300 5100
+	1    0    0    -1
+$EndComp
+NoConn ~ 6350 4850
+NoConn ~ 6400 4850
+NoConn ~ 6400 4900
+NoConn ~ 6350 4900
+NoConn ~ 6350 4950
+NoConn ~ 6400 4950
+NoConn ~ 6400 5000
+NoConn ~ 6350 5000
+NoConn ~ 6350 5050
+NoConn ~ 6400 5050
 $EndSCHEMATC

Commit message: PCB-V5 update
Panelization v1
Parts:
- removed e1: 02x06_pad, pcb-v5:02x06_pad, symbol sensOCampus:02x06_pad
Connections:
- no-connect marks 30 -> 20
Changed lines of the file:
@@
 Wire Notes Line
 	6300 1650 6300 450
-$Comp
-L sensOCampus:02x06_pad e1
-U 1 1 601241B4
-P 6300 5100
-F 0 "e1" H 6375 5575 50  0000 C CNN
-F 1 "02x06_pad" H 6375 5484 50  0000 C CNN
-F 2 "pcb-v5:02x06_pad" H 6300 5100 50  0001 C CNN
-F 3 "" H 6300 5100 50  0001 C CNN
-	1    6300 5100
-	1    0    0    -1
-$EndComp
-NoConn ~ 6350 4850
-NoConn ~ 6400 4850
-NoConn ~ 6400 4900
-NoConn ~ 6350 4900
-NoConn ~ 6350 4950
-NoConn ~ 6400 4950
-NoConn ~ 6400 5000
-NoConn ~ 6350 5000
-NoConn ~ 6350 5050
-NoConn ~ 6400 5050
 $EndSCHEMATC
