File: pcb/pcb-v5/panelized_v5.0.1.kicad_pcb (KiCad board)
At the start: 2 copper layers, 99.4 x 99.8 mm, 19 parts, among them J1 Conn_01x05_Female, J2 Conn_01x05_Female, J3 Conn_01x05_Female, J4 Conn_01x05_Male, Q1 2N7002, U1 AMS1117-3.3

Commit message: resistance+M2SIAME
Parts:
- removed the C1 at (127.4, 120.3)
- removed the C1 at (77.5, 120.3)
- removed the H2 at (123.1, 84.7)
- removed the J2 at (159.1, 82.3)
- removed the J4 at (156.6, 129.0)
- removed the Q1 at (123.8, 117.4)
- removed the REF** at (140.8, 106.4)
- removed the U1 at (124.3, 126.1)
- added C1: 10µF, Capacitor_SMD:C_0805_2012Metric_Pad1.18x1.45mm_HandSolder, F.Cu at (108.8, 122.1)
- added ESP1: ESP32, pcb-v5:ESP32_30_pins, F.Cu at (156.0, 87.0)
- added ESP1: ESP32, pcb-v5:ESP32_30_pins, F.Cu at (112.6, 117.5)
- added H2: MountingHole_Pad, MountingHole:MountingHole_3.2mm_M3_Pad, F.Cu at (164.8, 126.4)
- added H2: MountingHole_Pad, MountingHole:MountingHole_3.2mm_M3_Pad, F.Cu at (73.2, 126.4)
- added J2: Conn_01x05_Female, Connector_PinHeader_2.54mm:PinHeader_1x05_P2.54mm_Vertical, F.Cu at (128.8, 128.8)
- added J2: Conn_01x05_Female, Connector_PinHeader_2.54mm:PinHeader_1x05_P2.54mm_Vertical, F.Cu at (104.2, 128.9)
- added J4: Conn_01x05_Male, Connector_PinHeader_2.54mm:PinHeader_1x05_P2.54mm_Vertical, F.Cu at (131.3, 82.0)
- added J4: Conn_01x05_Male, Connector_PinHeader_2.54mm:PinHeader_1x05_P2.54mm_Vertical, F.Cu at (117.7, 92.1)
- added Q1: 2N7002, Package_TO_SOT_SMD:SOT-23, F.Cu at (164.1, 93.7)
- added Q1: 2N7002, Package_TO_SOT_SMD:SOT-23, F.Cu at (71.5, 114.7)
- added R2: 15k, Resistor_SMD:R_0805_2012Metric_Pad1.20x1.40mm_HandSolder, F.Cu at (163.3, 97.5)
- added R2: 15k, Resistor_SMD:R_0805_2012Metric_Pad1.20x1.40mm_HandSolder, F.Cu at (74.5, 112.7)
- added R3: 68, Resistor_SMD:R_0805_2012Metric_Pad1.20x1.40mm_HandSolder, F.Cu at (161.3, 95.0)
- added R3: 68, Resistor_SMD:R_0805_2012Metric_Pad1.20x1.40mm_HandSolder, F.Cu at (71.5, 119.8)
- added R4: 220, Resistor_SMD:R_0805_2012Metric_Pad1.20x1.40mm_HandSolder, B.Cu at (136.2, 102.4)
- added R4: 220, Resistor_SMD:R_0805_2012Metric_Pad1.20x1.40mm_HandSolder, B.Cu at (97.4, 95.9)
- added R4: 220, Resistor_SMD:R_0805_2012Metric_Pad1.20x1.40mm_HandSolder, B.Cu at (97.4, 45.6)
- added RE: 220, Resistor_SMD:R_0805_2012Metric_Pad1.20x1.40mm_HandSolder, B.Cu at (99.9, 95.9)
- added RE: 220, Resistor_SMD:R_0805_2012Metric_Pad1.20x1.40mm_HandSolder, B.Cu at (99.9, 45.6)
- added Re: 220, Resistor_SMD:R_0805_2012Metric_Pad1.20x1.40mm_HandSolder, B.Cu at (135.3, 99.5)
- added SW1: G71Y, pcb-v5:G71Y_µsw_smd, B.Cu at (168.7, 106.9)
- added SW1: G71Y, pcb-v5:G71Y_µsw_smd, B.Cu at (69.4, 86.1)
- added SW2: G71Y, pcb-v5:G71Y_µsw_smd, B.Cu at (168.7, 117.1)
- added SW2: G71Y, pcb-v5:G71Y_µsw_smd, B.Cu at (69.4, 96.4)
- added SW3: G71Y, pcb-v5:G71Y_µsw_smd, B.Cu at (69.4, 106.7)
- added U1: AMS1117-3.3, Package_TO_SOT_SMD:SOT-223-3_TabPin2, F.Cu at (163.6, 85.0)
- added U1: AMS1117-3.3, Package_TO_SOT_SMD:SOT-223-3_TabPin2, F.Cu at (114.6, 125.1)
- moved H1 61.7 mm to (115.2, 87.0), turned to 90 degrees
- moved OLED1 48.1 mm to (127.5, 123.1), turned to 90 degrees
- moved Q1 46.8 mm to (164.1, 43.4), turned to 180 degrees
- moved J1 46.5 mm to (144.1, 128.8), turned to 90 degrees
- moved R2 41.9 mm to (163.3, 47.2), turned to 270 degrees
- moved R3 40.6 mm to (161.3, 44.7), turned to 90 degrees
- moved R1 36.3 mm to (161.8, 52.0), turned to 90 degrees
- moved J3 33.6 mm to (117.7, 107.3), turned to 0 degrees
- moved OLED1 33.4 mm to (77.1, 38.7), turned to 0 degrees
- moved R1 29.7 mm to (73.3, 108.6), turned to 180 degrees
- moved REF** 4.58 mm to (92.0, 52.7), turned to 90 degrees
Other:
- board text added: "M2 SIAME"
