File: pcb/pcb-v5/pcb-v5.kicad_pcb (KiCad board)
At the start: 2 copper layers, 14 parts, among them J1 Conn_01x05_Female, J2 Conn_01x05_Female, J3 Conn_01x05_Female, J4 Conn_01x05_Male, SW1 G71Y, SW2 G71Y, SW3 G71Y, U1 AMS1117-3.3

Commit message: PCB-V5 update
Panelization v1
Parts:
- removed C1: 10µF, Capacitor_SMD:C_0805_2012Metric_Pad1.18x1.45mm_HandSolder
- removed D1: LED, LED_SMD:LED_0805_2012Metric_Pad1.15x1.40mm_HandSolder
- removed ESP1: ESP32, pcb-v5:ESP32_30_pins
- removed H1, H2: MountingHole_Pad, MountingHole:MountingHole_3.2mm_M3_Pad
- removed J1, J2, J3: Conn_01x05_Female, Connector_PinHeader_2.54mm:PinHeader_1x05_P2.54mm_Vertical
- removed J4: Conn_01x05_Male, Connector_PinHeader_2.54mm:PinHeader_1x05_P2.54mm_Vertical
- removed SW1, SW2, SW3: G71Y, pcb-v5:G71Y_µsw_smd
- removed U1: AMS1117-3.3, Package_TO_SOT_SMD:SOT-223-3_TabPin2

Commit message: PCB-V2 update
Added OSHW logo on both boards.
Upgraded power lines size to 0.6604.
Added every needed screen printings (VCC,SDA,SCL,...)
Parts:
- added REF**: OSHW-Logo2_9.8x8mm_SilkScreen, Symbol:OSHW-Logo2_9.8x8mm_SilkScreen, F.Cu at (154.2, 83.6)

Commit message: resistance+M2SIAME
Parts:
- added R4: 220, Resistor_SMD:R_0805_2012Metric_Pad1.20x1.40mm_HandSolder, B.Cu at (161.3, 88.9)
- added RE: 220, Resistor_SMD:R_0805_2012Metric_Pad1.20x1.40mm_HandSolder, B.Cu at (161.3, 91.4)
