File: pcb/pcb-v5/pcb-v5_buttons_top.kicad_pcb (KiCad board)
At the start: 2 copper layers, 15 parts, among them J1 Conn_01x05_Female, J2 Conn_01x05_Female, J3 Conn_01x05_Female, J4 Conn_01x05_Male, SW1 G71Y, SW2 G71Y, SW3 G71Y, U1 AMS1117-3.3

Commit message: resistance+M2SIAME
Parts:
- added R4: 220, Resistor_SMD:R_0805_2012Metric_Pad1.20x1.40mm_HandSolder, B.Cu at (159.4, 88.7)
- added Re: 220, Resistor_SMD:R_0805_2012Metric_Pad1.20x1.40mm_HandSolder, B.Cu at (160.3, 91.6)
